File: KiCad/IR_UART/IR_UART.kicad_pcb (KiCad board)
At the start: 2 copper layers, 21 x 36 mm, 23 parts, among them J1 Conn_01x04, J2 Mounting PTH, J3 Mounting PTH, J4 Mounting PTH, J5 Mounting PTH, Q1 BC817, U1 TSDP34156, U2 74HC132

Commit message: Update the schematic and the PCB
- Use 4.7k resistor instead of 6.8k in the timing circuit
- Minor changes to the board, mainly aroung the 4-pin connector
Parts:
- R4: value 600 -> 560
- R7: value 6.8k -> 4.7k
- moved J1 7.63 mm to (111.2, 74.6), turned to 90 degrees
Connections:
- J1 pad 1: +3.3V -> GND
- J1 pad 2: /EXT_TX -> /EXT_RX
- J1 pad 3: /EXT_RX -> /EXT_TX
- J1 pad 4: GND -> +3.3V
Routing:
- net /EXT_TX: track 17.7 -> 18.4 mm
- net /EXT_RX: track 47.4 -> 48.0 mm
- net +3.3V: track 49.9 -> 50.6 mm
